File: stm32c0_fdcan_module.kicad_sch (KiCad schematic)
At the start: 32 parts, among them IC1 STM32C092GCU6, IC2 TJA1051TK_3,118, J1 12505WS-04, J2 Conn_01x10, J3 Conn_01x10, J4 12505WS-06, SW1 DSHP02TSGER, U1 XC6206P332MR, Y1 8MHz_50X32mm

Commit message: 단면 배치 버전
Connections:
- net +3.3V: now also J2.1 (Pin_1)
- net 5V: no longer J2.1 (Pin_1), J2.2 (Pin_2)
- net GND: now also J2.2 (Pin_2)
Changed lines of the file:
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@@
 	)
 	(junction
-		(at 199.39 130.81)
-		(diameter 0)
-		(color 0 0 0 0)
-	)
-	(junction
 		(at 125.73 153.67)
 		(diameter 0)
@@
 	)
 	(junction
+		(at 199.39 153.67)
+		(diameter 0)
+		(color 0 0 0 0)
+	)
+	(junction
 		(at 204.47 96.52)
 		(diameter 0)
@@
 	(wire
 		(pts
+			(xy 199.39 133.35) (xy 199.39 153.67)
+		)
+		(stroke
+			(width 0)
+			(type default)
+		)
+	)
+	(wire
+		(pts
 			(xy 162.56 166.37) (xy 162.56 161.29)
 		)
@@
 	(wire
 		(pts
+			(xy 199.39 130.81) (xy 199.39 129.54)
+		)
+		(stroke
+			(width 0)
+			(type default)
+		)
+	)
+	(wire
+		(pts
 			(xy 36.83 162.56) (xy 63.5 162.56)
 		)
@@
 	(wire
 		(pts
-			(xy 199.39 148.59) (xy 200.66 148.59)
+			(xy 196.85 148.59) (xy 200.66 148.59)
 		)
 		(stroke
@@
 	(wire
 		(pts
-			(xy 199.39 138.43) (xy 200.66 138.43)
+			(xy 196.85 138.43) (xy 200.66 138.43)
 		)
 		(stroke
@@
 	(wire
 		(pts
-			(xy 199.39 140.97) (xy 200.66 140.97)
+			(xy 196.85 140.97) (xy 200.66 140.97)
 		)
 		(stroke
@@
 	(wire
 		(pts
-			(xy 199.39 143.51) (xy 200.66 143.51)
+			(xy 196.85 143.51) (xy 200.66 143.51)
 		)
 		(stroke
@@
 	(wire
 		(pts
-			(xy 199.39 151.13) (xy 200.66 151.13)
+			(xy 196.85 151.13) (xy 200.66 151.13)
 		)
 		(stroke
@@
 	(wire
 		(pts
-			(xy 199.39 130.81) (xy 200.66 130.81)
-		)
-		(stroke
-			(width 0)
-			(type default)
-		)
-	)
-	(wire
-		(pts
 			(xy 27.94 41.91) (xy 27.94 66.04)
 		)
@@
 	(wire
 		(pts
-			(xy 199.39 129.54) (xy 199.39 130.81)
-		)
-		(stroke
-			(width 0)
-			(type default)
-		)
-	)
-	(wire
-		(pts
 			(xy 160.02 43.18) (xy 171.45 43.18)
 		)
@@
 	(wire
 		(pts
-			(xy 199.39 133.35) (xy 199.39 130.81)
+			(xy 226.06 143.51) (xy 222.25 143.51)
 		)
 		(stroke
@@
 	(wire
 		(pts
-			(xy 226.06 143.51) (xy 222.25 143.51)
+			(xy 208.28 39.37) (xy 209.55 39.37)
 		)
 		(stroke
@@
 	(wire
 		(pts
-			(xy 208.28 39.37) (xy 209.55 39.37)
+			(xy 200.66 130.81) (xy 199.39 130.81)
 		)
 		(stroke
@@
 	(wire
 		(pts
-			(xy 199.39 146.05) (xy 200.66 146.05)
+			(xy 196.85 146.05) (xy 200.66 146.05)
 		)
 		(stroke
@@
 	(wire
 		(pts
-			(xy 199.39 135.89) (xy 200.66 135.89)
+			(xy 196.85 135.89) (xy 200.66 135.89)
 		)
 		(stroke
@@
 	(global_label "PA3"
 		(shape input)
-		(at 199.39 135.89 180)
+		(at 196.85 135.89 180)
 		(fields_autoplaced yes)
 		(effects
@@
 		)
 		(property "Intersheetrefs" "${INTERSHEET_REFS}"
-			(at 193.6978 135.89 0)
+			(at 191.1578 135.89 0)
 			(effects
 				(font
@@
 	(global_label "PA4"
 		(shape input)
-		(at 199.39 138.43 180)
+		(at 196.85 138.43 180)
 		(fields_autoplaced yes)
 		(effects
@@
 		)
 		(property "Intersheetrefs" "${INTERSHEET_REFS}"
-			(at 193.6978 138.43 0)
+			(at 191.1578 138.43 0)
 			(effects
 				(font
@@
 	(global_label "PA8"
 		(shape input)
-		(at 199.39 148.59 180)
+		(at 196.85 148.59 180)
 		(fields_autoplaced yes)
 		(effects
@@
 		)
 		(property "Intersheetrefs" "${INTERSHEET_REFS}"
-			(at 193.6978 148.59 0)
+			(at 191.1578 148.59 0)
 			(effects
 				(font
@@
 	(global_label "PA5"
 		(shape input)
-		(at 199.39 140.97 180)
+		(at 196.85 140.97 180)
 		(fields_autoplaced yes)
 		(effects
@@
 		)
 		(property "Intersheetrefs" "${INTERSHEET_REFS}"
-			(at 193.6978 140.97 0)
+			(at 191.1578 140.97 0)
 			(effects
 				(font
@@
 	(global_label "PA7"
 		(shape input)
-		(at 199.39 146.05 180)
+		(at 196.85 146.05 180)
 		(fields_autoplaced yes)
 		(effects
@@
 		)
 		(property "Intersheetrefs" "${INTERSHEET_REFS}"
-			(at 193.6978 146.05 0)
+			(at 191.1578 146.05 0)
 			(effects
 				(font
@@
 	(global_label "PC6"
 		(shape input)
-		(at 199.39 151.13 180)
+		(at 196.85 151.13 180)
 		(fields_autoplaced yes)
 		(effects
@@
 		)
 		(property "Intersheetrefs" "${INTERSHEET_REFS}"
-			(at 193.6978 151.13 0)
+			(at 191.1578 151.13 0)
 			(effects
 				(font
@@
 	(global_label "PA6"
 		(shape input)
-		(at 199.39 143.51 180)
+		(at 196.85 143.51 180)
 		(fields_autoplaced yes)
 		(effects
@@
 		)
 		(property "Intersheetrefs" "${INTERSHEET_REFS}"
-			(at 193.6978 143.51 0)
+			(at 191.1578 143.51 0)
 			(effects
 				(font
@@
 	)
 	(symbol
-		(lib_id "power:VCC")
-		(at 199.39 129.54 0)
-		(unit 1)
-		(exclude_from_sim no)
-		(in_bom yes)
-		(on_board yes)
-		(dnp no)
-		(fields_autoplaced yes)
-		(property "Reference" "#PWR027"
-			(at 199.39 133.35 0)
-			(effects
-				(font
-					(size 1.27 1.27)
-				)
-				(hide yes)
-			)
-		)
-		(property "Value" "5V"
-			(at 199.39 124.46 0)
-			(effects
-				(font
-					(size 1.27 1.27)
-				)
-			)
-		)
-		(property "Footprint" ""
-			(at 199.39 129.54 0)
-			(effects
-				(font
-					(size 1.27 1.27)
-				)
-				(hide yes)
-			)
-		)
-		(property "Datasheet" ""
-			(at 199.39 129.54 0)
-			(effects
-				(font
-					(size 1.27 1.27)
-				)
-				(hide yes)
-			)
-		)
-		(property "Description" "Power symbol creates a global label with name \"VCC\""
-			(at 199.39 129.54 0)
-			(effects
-				(font
-					(size 1.27 1.27)
-				)
-				(hide yes)
-			)
-		)
-		(pin "1"
-		)
-		(instances
-			(project "stm32c0_fdcan_module"
-				(path "/783957ae-1b6b-407f-8046-ed2eea5bf45d"
-					(reference "#PWR027")
-					(unit 1)
-				)
-			)
-		)
-	)
-	(symbol
 		(lib_id "TJA1051TK_3_118:TJA1051TK_3,118")
 		(at 171.45 35.56 0)
@@
 					(unit 1)
 				)
+			)
+		)
+	)
+	(symbol
+		(lib_id "power:+3.3V")
+		(at 199.39 129.54 0)
+		(unit 1)
+		(exclude_from_sim no)
+		(in_bom yes)
+		(on_board yes)
+		(dnp no)
+		(fields_autoplaced yes)
+		(property "Reference" "#PWR026"
+			(at 199.39 133.35 0)
+			(effects
+				(font
+					(size 1.27 1.27)
+				)
+				(hide yes)
+			)
+		)
+		(property "Value" "+3.3V"
+			(at 199.39 124.46 0)
+			(effects
+				(font
+					(size 1.27 1.27)
+				)
+			)
+		)
+		(property "Footprint" ""
+			(at 199.39 129.54 0)
+			(effects
+				(font
+					(size 1.27 1.27)
+				)
+				(hide yes)
+			)
+		)
+		(property "Datasheet" ""
+			(at 199.39 129.54 0)
+			(effects
+				(font
+					(size 1.27 1.27)
+				)
+				(hide yes)
+			)
+		)
+		(property "Description" "Power symbol creates a global label with name \"+3.3V\""
+			(at 199.39 129.54 0)
+			(effects
+				(font
+					(size 1.27 1.27)
+				)
+				(hide yes)
+			)
+		)
+		(pin "1"
+		)
+		(instances
+			(project "stm32c0_fdcan_module"
+				(path "/783957ae-1b6b-407f-8046-ed2eea5bf45d"
+					(reference "#PWR026")
+					(unit 1)
+				)
